File: hogefuga.sch (KiCad schematic (older format))
At the start: 41 parts, among them J1 MJ-4PP-9, SW1 SW_PUSH, SW10 SW_PUSH, SW11 SW_PUSH, SW12 SW_PUSH, SW13 SW_PUSH, SW14 SW_PUSH, SW15 SW_PUSH, SW16 SW_PUSH, SW17 SW_PUSH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

Commit message: rev0.2
Parts:
- SW1, SW10, SW11, SW12, SW13, SW14, SW15, SW2, SW3, SW4, SW5, SW6, SW7, SW8, SW9: footprint lib:SW_Matias_1.00u -> keyboard_parts:ALPS_SKCM
Changed lines of the file:
@@
 F 0 "SW1" H 5600 1805 50  0000 C CNN
 F 1 "SW_PUSH" H 5600 1714 50  0000 C CNN
-F 2 "lib:SW_Matias_1.00u" H 5600 1550 50  0001 C CNN
+F 2 "keyboard_parts:ALPS_SKCM" H 5600 1550 50  0001 C CNN
 F 3 "" H 5600 1550 50  0000 C CNN
 	1    5600 1550
@@
 F 0 "SW2" H 6650 1805 50  0000 C CNN
 F 1 "SW_PUSH" H 6650 1714 50  0000 C CNN
-F 2 "lib:SW_Matias_1.00u" H 6650 1550 50  0001 C CNN
+F 2 "keyboard_parts:ALPS_SKCM" H 6650 1550 50  0001 C CNN
 F 3 "" H 6650 1550 50  0000 C CNN
 	1    6650 1550
@@
 F 0 "SW3" H 7750 1805 50  0000 C CNN
 F 1 "SW_PUSH" H 7750 1714 50  0000 C CNN
-F 2 "lib:SW_Matias_1.00u" H 7750 1550 50  0001 C CNN
+F 2 "keyboard_parts:ALPS_SKCM" H 7750 1550 50  0001 C CNN
 F 3 "" H 7750 1550 50  0000 C CNN
 	1    7750 1550
@@
 F 0 "SW4" H 8800 1805 50  0000 C CNN
 F 1 "SW_PUSH" H 8800 1714 50  0000 C CNN
-F 2 "lib:SW_Matias_1.00u" H 8800 1550 50  0001 C CNN
+F 2 "keyboard_parts:ALPS_SKCM" H 8800 1550 50  0001 C CNN
 F 3 "" H 8800 1550 50  0000 C CNN
 	1    8800 1550
@@
 F 0 "SW5" H 9850 1805 50  0000 C CNN
 F 1 "SW_PUSH" H 9850 1714 50  0000 C CNN
-F 2 "lib:SW_Matias_1.00u" H 9850 1550 50  0001 C CNN
+F 2 "keyboard_parts:ALPS_SKCM" H 9850 1550 50  0001 C CNN
 F 3 "" H 9850 1550 50  0000 C CNN
 	1    9850 1550
@@
 F 0 "SW6" H 5600 2305 50  0000 C CNN
 F 1 "SW_PUSH" H 5600 2214 50  0000 C CNN
-F 2 "lib:SW_Matias_1.00u" H 5600 2050 50  0001 C CNN
+F 2 "keyboard_parts:ALPS_SKCM" H 5600 2050 50  0001 C CNN
 F 3 "" H 5600 2050 50  0000 C CNN
 	1    5600 2050
@@
 F 0 "SW7" H 6650 2305 50  0000 C CNN
 F 1 "SW_PUSH" H 6650 2214 50  0000 C CNN
-F 2 "lib:SW_Matias_1.00u" H 6650 2050 50  0001 C CNN
+F 2 "keyboard_parts:ALPS_SKCM" H 6650 2050 50  0001 C CNN
 F 3 "" H 6650 2050 50  0000 C CNN
 	1    6650 2050
@@
 F 0 "SW8" H 7750 2305 50  0000 C CNN
 F 1 "SW_PUSH" H 7750 2214 50  0000 C CNN
-F 2 "lib:SW_Matias_1.00u" H 7750 2050 50  0001 C CNN
+F 2 "keyboard_parts:ALPS_SKCM" H 7750 2050 50  0001 C CNN
 F 3 "" H 7750 2050 50  0000 C CNN
 	1    7750 2050
@@
 F 0 "SW9" H 8800 2305 50  0000 C CNN
 F 1 "SW_PUSH" H 8800 2214 50  0000 C CNN
-F 2 "lib:SW_Matias_1.00u" H 8800 2050 50  0001 C CNN
+F 2 "keyboard_parts:ALPS_SKCM" H 8800 2050 50  0001 C CNN
 F 3 "" H 8800 2050 50  0000 C CNN
 	1    8800 2050
@@
 F 0 "SW10" H 9850 2305 50  0000 C CNN
 F 1 "SW_PUSH" H 9850 2214 50  0000 C CNN
-F 2 "lib:SW_Matias_1.00u" H 9850 2050 50  0001 C CNN
+F 2 "keyboard_parts:ALPS_SKCM" H 9850 2050 50  0001 C CNN
 F 3 "" H 9850 2050 50  0000 C CNN
 	1    9850 2050
@@
 F 0 "SW11" H 5600 2805 50  0000 C CNN
 F 1 "SW_PUSH" H 5600 2714 50  0000 C CNN
-F 2 "lib:SW_Matias_1.00u" H 5600 2550 50  0001 C CNN
+F 2 "keyboard_parts:ALPS_SKCM" H 5600 2550 50  0001 C CNN
 F 3 "" H 5600 2550 50  0000 C CNN
 	1    5600 2550
@@
 F 0 "SW12" H 6650 2805 50  0000 C CNN
 F 1 "SW_PUSH" H 6650 2714 50  0000 C CNN
-F 2 "lib:SW_Matias_1.00u" H 6650 2550 50  0001 C CNN
+F 2 "keyboard_parts:ALPS_SKCM" H 6650 2550 50  0001 C CNN
 F 3 "" H 6650 2550 50  0000 C CNN
 	1    6650 2550
@@
 F 0 "SW13" H 7750 2805 50  0000 C CNN
 F 1 "SW_PUSH" H 7750 2714 50  0000 C CNN
-F 2 "lib:SW_Matias_1.00u" H 7750 2550 50  0001 C CNN
+F 2 "keyboard_parts:ALPS_SKCM" H 7750 2550 50  0001 C CNN
 F 3 "" H 7750 2550 50  0000 C CNN
 	1    7750 2550
@@
 F 0 "SW14" H 8800 2805 50  0000 C CNN
 F 1 "SW_PUSH" H 8800 2714 50  0000 C CNN
-F 2 "lib:SW_Matias_1.00u" H 8800 2550 50  0001 C CNN
+F 2 "keyboard_parts:ALPS_SKCM" H 8800 2550 50  0001 C CNN
 F 3 "" H 8800 2550 50  0000 C CNN
 	1    8800 2550
@@
 F 0 "SW15" H 9850 2805 50  0000 C CNN
 F 1 "SW_PUSH" H 9850 2714 50  0000 C CNN
-F 2 "lib:SW_Matias_1.00u" H 9850 2550 50  0001 C CNN
+F 2 "keyboard_parts:ALPS_SKCM" H 9850 2550 50  0001 C CNN
 F 3 "" H 9850 2550 50  0000 C CNN
 	1    9850 2550
@@
 	9550 2000 9550 2050
 Wire Wire Line
-	5250 1000 5250 1550
-Wire Wire Line
 	7450 1000 7450 1550
 Wire Wire Line
@@
 Wire Wire Line
 	5250 1550 5250 2050
+Wire Wire Line
+	5250 1000 5250 1550
 $EndSCHEMATC

Commit message: スイッチを全てtmkさんのフットプリントに変更
Parts:
- SW16, SW17, SW18, SW19: footprint lib:SW_Matias_1.25u -> keyboard_parts:ALPS_SKCM
Changed lines of the file:
@@
 Text GLabel 4850 2850 0    50   Input ~ 0
 row2
-Text GLabel 4900 3350 0    50   Input ~ 0
+Text GLabel 4900 3600 0    50   Input ~ 0
 row3
 Wire Wire Line
@@
 Connection ~ 8050 1850
 Wire Wire Line
-	4900 3350 5900 3350
+	4900 3600 5900 3600
 Text GLabel 1900 2200 0    50   Input ~ 0
 row0
@@
 	6950 2850 8050 2850
 Connection ~ 9100 2850
-Wire Wire Line
-	8050 2850 9100 2850
 Connection ~ 8050 2850
 Wire Wire Line
@@
 L kbd:SW_PUSH SW16
 U 1 1 5BC237A6
-P 5600 3050
-F 0 "SW16" H 5600 3305 50  0000 C CNN
-F 1 "SW_PUSH" H 5600 3214 50  0000 C CNN
-F 2 "lib:SW_Matias_1.25u" H 5600 3050 50  0001 C CNN
-F 3 "" H 5600 3050 50  0000 C CNN
-	1    5600 3050
-	-1   0    0    1
+P 5600 3300
+F 0 "SW16" H 5600 3555 50  0000 C CNN
+F 1 "SW_PUSH" H 5600 3464 50  0000 C CNN
+F 2 "keyboard_parts:ALPS_SKCM" H 5600 3300 50  0001 C CNN
+F 3 "" H 5600 3300 50  0000 C CNN
+	1    5600 3300
+	1    0    0    -1
 $EndComp
 $Comp
 L Device:D D16
 U 1 1 5BC237AC
-P 5900 3200
-F 0 "D16" V 5946 3121 50  0000 R CNN
-F 1 "D" V 5855 3121 50  0000 R CNN
-F 2 "kbd:D3_TH_SMD" H 5900 3200 50  0001 C CNN
-F 3 "~" H 5900 3200 50  0001 C CNN
-	1    5900 3200
+P 5900 3450
+F 0 "D16" V 5946 3371 50  0000 R CNN
+F 1 "D" V 5855 3371 50  0000 R CNN
+F 2 "kbd:D3_TH_SMD" H 5900 3450 50  0001 C CNN
+F 3 "~" H 5900 3450 50  0001 C CNN
+	1    5900 3450
 	0    -1   -1   0
 $EndComp
@@
 L kbd:SW_PUSH SW17
 U 1 1 5BC237B2
-P 6650 3050
-F 0 "SW17" H 6650 3305 50  0000 C CNN
-F 1 "SW_PUSH" H 6650 3214 50  0000 C CNN
-F 2 "lib:SW_Matias_1.25u" H 6650 3050 50  0001 C CNN
-F 3 "" H 6650 3050 50  0000 C CNN
-	1    6650 3050
-	-1   0    0    1
+P 6650 3300
+F 0 "SW17" H 6650 3555 50  0000 C CNN
+F 1 "SW_PUSH" H 6650 3464 50  0000 C CNN
+F 2 "keyboard_parts:ALPS_SKCM" H 6650 3300 50  0001 C CNN
+F 3 "" H 6650 3300 50  0000 C CNN
+	1    6650 3300
+	1    0    0    -1
 $EndComp
 $Comp
 L Device:D D17
 U 1 1 5BC237B8
-P 6950 3200
-F 0 "D17" V 6996 3121 50  0000 R CNN
-F 1 "D" V 6905 3121 50  0000 R CNN
-F 2 "kbd:D3_TH_SMD" H 6950 3200 50  0001 C CNN
-F 3 "~" H 6950 3200 50  0001 C CNN
-	1    6950 3200
+P 6950 3450
+F 0 "D17" V 6996 3371 50  0000 R CNN
+F 1 "D" V 6905 3371 50  0000 R CNN
+F 2 "kbd:D3_TH_SMD" H 6950 3450 50  0001 C CNN
+F 3 "~" H 6950 3450 50  0001 C CNN
+	1    6950 3450
 	0    -1   -1   0
 $EndComp
@@
 L kbd:SW_PUSH SW18
 U 1 1 5BC237CA
-P 8800 3050
-F 0 "SW18" H 8800 3305 50  0000 C CNN
-F 1 "SW_PUSH" H 8800 3214 50  0000 C CNN
-F 2 "lib:SW_Matias_1.25u" H 8800 3050 50  0001 C CNN
-F 3 "" H 8800 3050 50  0000 C CNN
-	1    8800 3050
+P 8800 3300
+F 0 "SW18" H 8800 3555 50  0000 C CNN
+F 1 "SW_PUSH" H 8800 3464 50  0000 C CNN
+F 2 "keyboard_parts:ALPS_SKCM" H 8800 3300 50  0001 C CNN
+F 3 "" H 8800 3300 50  0000 C CNN
+	1    8800 3300
 	-1   0    0    1
 $EndComp
@@
 L Device:D D18
 U 1 1 5BC237D0
-P 9100 3200
-F 0 "D18" V 9146 3121 50  0000 R CNN
-F 1 "D" V 9055 3121 50  0000 R CNN
-F 2 "kbd:D3_TH_SMD" H 9100 3200 50  0001 C CNN
-F 3 "~" H 9100 3200 50  0001 C CNN
-	1    9100 3200
+P 9100 3450
+F 0 "D18" V 9146 3371 50  0000 R CNN
+F 1 "D" V 9055 3371 50  0000 R CNN
+F 2 "kbd:D3_TH_SMD" H 9100 3450 50  0001 C CNN
+F 3 "~" H 9100 3450 50  0001 C CNN
+	1    9100 3450
 	0    -1   -1   0
 $EndComp
@@
 L kbd:SW_PUSH SW19
 U 1 1 5BC237D6
-P 9850 3050
-F 0 "SW19" H 9850 3305 50  0000 C CNN
-F 1 "SW_PUSH" H 9850 3214 50  0000 C CNN
-F 2 "lib:SW_Matias_1.25u" H 9850 3050 50  0001 C CNN
-F 3 "" H 9850 3050 50  0000 C CNN
-	1    9850 3050
+P 9850 3300
+F 0 "SW19" H 9850 3555 50  0000 C CNN
+F 1 "SW_PUSH" H 9850 3464 50  0000 C CNN
+F 2 "keyboard_parts:ALPS_SKCM" H 9850 3300 50  0001 C CNN
+F 3 "" H 9850 3300 50  0000 C CNN
+	1    9850 3300
 	-1   0    0    1
 $EndComp
@@
 L Device:D D19
 U 1 1 5BC237DC
-P 10150 3200
-F 0 "D19" V 10196 3121 50  0000 R CNN
-F 1 "D" V 10105 3121 50  0000 R CNN
-F 2 "kbd:D3_TH_SMD" H 10150 3200 50  0001 C CNN
-F 3 "~" H 10150 3200 50  0001 C CNN
-	1    10150 3200
-	0    -1   -1   0
-$EndComp
-Wire Wire Line
-	5250 3050 5300 3050
-Wire Wire Line
-	6350 3050 6300 3050
-Connection ~ 5900 3350
-Connection ~ 6950 3350
-Connection ~ 9100 3350
-Wire Wire Line
-	5900 3350 6950 3350
-Wire Wire Line
-	9100 3350 10150 3350
+P 10150 3450
+F 0 "D19" V 10196 3371 50  0000 R CNN
+F 1 "D" V 10105 3371 50  0000 R CNN
+F 2 "kbd:D3_TH_SMD" H 10150 3450 50  0001 C CNN
+F 3 "~" H 10150 3450 50  0001 C CNN
+	1    10150 3450
+	0    -1   -1   0
+$EndComp
+Wire Wire Line
+	5250 3300 5300 3300
+Wire Wire Line
+	6350 3300 6300 3300
+Connection ~ 5900 3600
+Connection ~ 6950 3600
+Connection ~ 9100 3600
+Wire Wire Line
+	5900 3600 6950 3600
 Connection ~ 5250 2050
+Connection ~ 6300 2050
+Connection ~ 7450 2050
+Wire Wire Line
+	7450 2050 7450 2550
+Connection ~ 8500 2050
+Connection ~ 9550 2050
+Wire Wire Line
+	5250 2000 5250 2050
+Wire Wire Line
+	7450 2000 7450 2050
+Wire Wire Line
+	8500 2000 8500 2050
+Wire Wire Line
+	9550 2000 9550 2050
+Wire Wire Line
+	7450 1000 7450 1550
+Wire Wire Line
+	8500 1000 8500 1550
+Wire Wire Line
+	9550 1000 9550 1550
+Wire Wire Line
+	6300 2000 6300 2050
+Wire Wire Line
+	6300 1000 6300 1550
+Wire Wire Line
+	4850 2350 5900 2350
+Wire Wire Line
+	4850 2850 5900 2850
+Connection ~ 9550 1550
+Wire Wire Line
+	9550 1550 9550 2050
+Connection ~ 8500 1550
+Wire Wire Line
+	8500 1550 8500 2050
+Connection ~ 7450 1550
+Wire Wire Line
+	7450 1550 7450 2050
+Connection ~ 6300 1550
+Wire Wire Line
+	6300 1550 6300 2050
+Connection ~ 5250 1550
+Wire Wire Line
+	5250 1550 5250 2050
+Wire Wire Line
+	5250 1000 5250 1550
+Wire Wire Line
+	8050 2850 9100 2850
+Wire Wire Line
+	8500 2050 8500 2550
+Connection ~ 8500 2550
+Wire Wire Line
+	8500 2550 8500 3300
+Wire Wire Line
+	9550 2050 9550 2550
+Connection ~ 9550 2550
+Wire Wire Line
+	9550 2550 9550 3300
+Wire Wire Line
+	6300 2050 6300 2550
+Connection ~ 6300 2550
+Wire Wire Line
+	6300 2550 6300 3300
 Wire Wire Line
 	5250 2050 5250 2550
 Connection ~ 5250 2550
 Wire Wire Line
-	5250 2550 5250 3050
-Connection ~ 6300 2050
-Connection ~ 6300 2550
-Wire Wire Line
-	6300 2550 6300 3050
-Connection ~ 7450 2050
-Wire Wire Line
-	7450 2050 7450 2550
-Connection ~ 8500 2050
-Wire Wire Line
-	8500 2050 8500 2550
-Connection ~ 8500 2550
-Wire Wire Line
-	8500 2550 8500 3050
-Connection ~ 9550 2050
-Wire Wire Line
-	9550 2050 9550 2550
-Connection ~ 9550 2550
-Wire Wire Line
-	9550 2550 9550 3050
-Wire Wire Line
-	6950 3350 9100 3350
-Wire Wire Line
-	5250 2000 5250 2050
-Wire Wire Line
-	7450 2000 7450 2050
-Wire Wire Line
-	8500 2000 8500 2050
-Wire Wire Line
-	9550 2000 9550 2050
-Wire Wire Line
-	7450 1000 7450 1550
-Wire Wire Line
-	8500 1000 8500 1550
-Wire Wire Line
-	9550 1000 9550 1550
-Wire Wire Line
-	6300 2050 6300 2550
-Wire Wire Line
-	6300 2000 6300 2050
-Wire Wire Line
-	6300 1000 6300 1550
-Wire Wire Line
-	4850 2350 5900 2350
-Wire Wire Line
-	4850 2850 5900 2850
-Connection ~ 9550 1550
-Wire Wire Line
-	9550 1550 9550 2050
-Connection ~ 8500 1550
-Wire Wire Line
-	8500 1550 8500 2050
-Connection ~ 7450 1550
-Wire Wire Line
-	7450 1550 7450 2050
-Connection ~ 6300 1550
-Wire Wire Line
-	6300 1550 6300 2050
-Connection ~ 5250 1550
-Wire Wire Line
-	5250 1550 5250 2050
-Wire Wire Line
-	5250 1000 5250 1550
+	5250 2550 5250 3300
+Wire Wire Line
+	6950 3600 9100 3600
+Wire Wire Line
+	9100 3600 10150 3600
 $EndSCHEMATC
